File: KiCad/Main/3X VCO.kicad_sch (KiCad schematic)
At the start: 92 parts, among them J1 Conn_01x32_Socket, J2 Conn_02x05_Odd_Even, J3 Conn_01x32_Socket, Q1 BC558, Q2 BC548, Q3 BC558, Q4 BC548, Q5 BC558, Q6 BC548, U1 40106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

Commit message: refactor: Change main schematic to Op-Amp per VCO. Add net labels for VCO outputs
Parts:
- added unit 4 of U4
- U2, U3, U4: footprint Package_DIP:DIP-14_W7.62mm_Socket -> (none)
Connections:
- net GND: now also U2.12 (+), U2.13 (-)
- net VCO3PwmPot1: now also U4.9 (-); no longer U2.6 (-)
- net VCO3WaveMixPot2: now also U4.12 (+); no longer U3.10 (+)
- net at C3.1, R16.2, U2.10 (+): now also U2.5 (+); no longer U3.5 (+)
- net at R18.1, R22.2: now also U2.6 (-); no longer U3.6 (-)
- net at R22.1, R24.2: now also U2.7; no longer U3.7
- net at R46.1, R48.1: now also U3.10 (+); no longer U4.10 (+)
- net at R46.2: now also U3.14; no longer U4.7
- net at C8.1, R43.2: now also U3.12 (+), U3.5 (+); no longer U4.3 (+), U4.5 (+)
- net at R41.1, R42.1, R44.1: now also U3.13 (-); no longer U4.6 (-)
- net at C2.1, D2.1 (K), Q4.1 (C)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: now also U4.3 (+); no longer U2.12 (+)
- net at U3.8, U3.9 (-): now also R50.2; no longer R33.2
- net at C7.1, D5.1 (K), Q6.1 (C)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: now also U3.3 (+); no longer U3.12 (+)
- net at R45.1, R47.2: now also U3.6 (-); no longer U4.2 (-)
- net at R47.1, R49.2: now also U3.7; no longer U4.1
- net at C4.1, R20.2: now also U4.10 (+), U4.5 (+); no longer U2.5 (+), U3.3 (+)
- net at R23.1, R27.2: now also U4.6 (-); no longer U3.2 (-)
- net at R27.1, R29.2: now also U4.7; no longer U3.1
- net at D4.2 (A), R19.1: now also U4.8; no longer U2.7
- new net: C8.2, U3.1, U3.2 (-)
- new net: C4.2, U4.1, U4.2 (-)
- new net: R33.2, U4.13 (-), U4.14
- now unconnected: U2.14
- no-connect marks 12 -> 13
Other:
- note removed: "PULSE OUT"
- note removed: "SAW OUT"
