File: KiCad/Main/MAIN.kicad_sch (KiCad schematic)
At the start: 92 parts, among them J1 Conn_01x32_Socket, J2 Conn_02x05_Odd_Even, J3 Conn_01x32_Socket, Q1 BC558, Q2 BC548, Q3 BC558, Q4 BC548, Q5 BC558, Q6 BC548, U1 40106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

Commit message: refactor: Rename KiCad files
Parts:
- U2, U3, U4: footprint (none) -> Package_DIP:DIP-14_W7.62mm_Socket
Changed lines of the file:
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@@
 			)
 		)
-		(property "Footprint" ""
+		(property "Footprint" "Package_DIP:DIP-14_W7.62mm_Socket"
 			(at 142.875 309.88 0)
 			(effects
@@
 			)
 		)
-		(property "Footprint" ""
+		(property "Footprint" "Package_DIP:DIP-14_W7.62mm_Socket"
 			(at 360.045 184.15 0)
 			(effects
@@
 			)
 		)
-		(property "Footprint" ""
+		(property "Footprint" "Package_DIP:DIP-14_W7.62mm_Socket"
 			(at 132.715 285.75 0)
 			(effects
@@
 			)
 		)
-		(property "Footprint" ""
+		(property "Footprint" "Package_DIP:DIP-14_W7.62mm_Socket"
 			(at 167.005 288.29 0)
 			(effects
@@
 			)
 		)
-		(property "Footprint" ""
+		(property "Footprint" "Package_DIP:DIP-14_W7.62mm_Socket"
 			(at 523.24 87.63 0)
 			(effects
@@
 			)
 		)
-		(property "Footprint" ""
+		(property "Footprint" "Package_DIP:DIP-14_W7.62mm_Socket"
 			(at 123.825 93.98 0)
 			(effects
@@
 			)
 		)
-		(property "Footprint" ""
+		(property "Footprint" "Package_DIP:DIP-14_W7.62mm_Socket"
 			(at 363.855 149.86 0)
 			(effects
@@
 			)
 		)
-		(property "Footprint" ""
+		(property "Footprint" "Package_DIP:DIP-14_W7.62mm_Socket"
 			(at 502.92 87.63 0)
 			(effects
@@
 			)
 		)
-		(property "Footprint" ""
+		(property "Footprint" "Package_DIP:DIP-14_W7.62mm_Socket"
 			(at 113.665 69.85 0)
 			(effects
@@
 			)
 		)
-		(property "Footprint" ""
+		(property "Footprint" "Package_DIP:DIP-14_W7.62mm_Socket"
 			(at 210.185 111.125 0)
 			(effects
@@
 			)
 		)
-		(property "Footprint" ""
+		(property "Footprint" "Package_DIP:DIP-14_W7.62mm_Socket"
 			(at 329.565 147.32 0)
 			(effects
@@
 			)
 		)
-		(property "Footprint" ""
+		(property "Footprint" "Package_DIP:DIP-14_W7.62mm_Socket"
 			(at 381.635 167.64 0)
 			(effects
@@
 			)
 		)
-		(property "Footprint" ""
+		(property "Footprint" "Package_DIP:DIP-14_W7.62mm_Socket"
 			(at 219.075 279.4 0)
 			(effects
@@
 			)
 		)
-		(property "Footprint" ""
+		(property "Footprint" "Package_DIP:DIP-14_W7.62mm_Socket"
 			(at 147.955 72.39 0)
 			(effects
@@
 			)
 		)
-		(property "Footprint" ""
+		(property "Footprint" "Package_DIP:DIP-14_W7.62mm_Socket"
 			(at 542.29 87.63 0)
 			(effects

Commit message: refactor: Rework Main board PCB
Changed lines of the file:
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@@
 (kicad_sch
-	(version 20231120)
+	(version 20250114)
 	(generator "eeschema")
-	(generator_version "8.0")
+	(generator_version "9.0")
 	(paper "A2")
+	(text "WAVE MIX"
+		(exclude_from_sim no)
+		(at 189.865 300.99 0)
+		(effects
+			(font
+				(size 1.27 1.27)
+				(italic yes)
+			)
+			(justify left bottom)
+		)
+	)
+	(text "COARSE"
+		(exclude_from_sim no)
+		(at 298.45 144.78 0)
+		(effects
+			(font
+				(size 1.27 1.27)
+				(italic yes)
+			)
+			(justify left bottom)
+		)
+	)
+	(text "VCO1"
+		(exclude_from_sim no)
+		(at 137.795 53.34 0)
+		(effects
+			(font
+				(size 2.9972 2.9972)
+				(thickness 0.5994)
+				(bold yes)
+			)
+			(justify right bottom)
+		)
+	)
+	(text "FINE"
+		(exclude_from_sim no)
+		(at 303.53 163.195 0)
+		(effects
+			(font
+				(size 1.27 1.27)
+				(italic yes)
+			)
+			(justify right bottom)
+		)
+	)
+	(text "COARSE"
+		(exclude_from_sim no)
+		(at 82.55 67.31 0)
+		(effects
+			(font
+				(size 1.27 1.27)
+				(italic yes)
+			)
+			(justify left bottom)
+		)
+	)
+	(text "VCO3\n"
+		(exclude_from_sim no)
+		(at 156.845 269.24 0)
+		(effects
+			(font
+				(size 2.9972 2.9972)
+				(thickness 0.5994)
+				(bold yes)
+			)
+			(justify right bottom)
+		)
+	)
+	(text "FINE"
+		(exclude_from_sim no)
+		(at 106.68 301.625 0)
+		(effects
+			(font
+				(size 1.27 1.27)
+				(italic yes)
+			)
+			(justify right bottom)
+		)
+	)
+	(text "IC POWER"
+		(exclude_from_sim no)
+		(at 509.27 77.47 0)
+		(effects
+			(font
+				(size 2.9972 2.9972)
+				(thickness 0.5994)
+				(bold yes)
+			)
+			(justify left bottom)
+		)
+	)
+	(text "FINE"
+		(exclude_from_sim no)
+		(at 87.63 85.725 0)
+		(effects
+			(font
+				(size 1.27 1.27)
+				(italic yes)
+			)
+			(justify right bottom)
+		)
+	)
+	(text "COARSE"
+		(exclude_from_sim no)
+		(at 101.6 283.21 0)
+		(effects
+			(font
+				(size 1.27 1.27)
+				(italic yes)
+			)
+			(justify left bottom)
+		)
+	)
+	(text "POWER HEADER"
+		(exclude_from_sim no)
+		(at 502.92 39.37 0)
+		(effects
+			(font
+				(size 2.9972 2.9972)
+				(thickness 0.5994)
+				(bold yes)
+			)
+			(justify left bottom)
+		)
+	)
+	(text "CONNECTORS\n"
+		(exclude_from_sim no)
+		(at 504.825 191.135 0)
+		(effects
+			(font
+				(size 2.9972 2.9972)
+				(thickness 0.5994)
+				(bold yes)
+			)
+			(justify left bottom)
+		)
+	)
+	(text "VCO2\n"
+		(exclude_from_sim no)
+		(at 353.695 130.81 0)
+		(effects
+			(font
+				(size 2.9972 2.9972)
+				(thickness 0.5994)
+				(bold yes)
+			)
+			(justify right bottom)
+		)
+	)
 	(junction
 		(at 200.025 312.42)
@@
 		)
 	)
-	(text "WAVE MIX"
-		(exclude_from_sim no)
-		(at 189.865 300.99 0)
-		(effects
-			(font
-				(size 1.27 1.27)
-				(italic yes)
-			)
-			(justify left bottom)
-		)
-	)
-	(text "COARSE"
-		(exclude_from_sim no)
-		(at 298.45 144.78 0)
-		(effects
-			(font
-				(size 1.27 1.27)
-				(italic yes)
-			)
-			(justify left bottom)
-		)
-	)
-	(text "VCO1"
-		(exclude_from_sim no)
-		(at 137.795 53.34 0)
-		(effects
-			(font
-				(size 2.9972 2.9972)
-				(thickness 0.5994)
-				(bold yes)
-			)
-			(justify right bottom)
-		)
-	)
-	(text "FINE"
-		(exclude_from_sim no)
-		(at 303.53 163.195 0)
-		(effects
-			(font
-				(size 1.27 1.27)
-				(italic yes)
-			)
-			(justify right bottom)
-		)
-	)
-	(text "COARSE"
-		(exclude_from_sim no)
-		(at 82.55 67.31 0)
-		(effects
-			(font
-				(size 1.27 1.27)
-				(italic yes)
-			)
-			(justify left bottom)
-		)
-	)
-	(text "VCO3\n"
-		(exclude_from_sim no)
-		(at 156.845 269.24 0)
-		(effects
-			(font
-				(size 2.9972 2.9972)
-				(thickness 0.5994)
-				(bold yes)
-			)
-			(justify right bottom)
-		)
-	)
-	(text "FINE"
-		(exclude_from_sim no)
-		(at 106.68 301.625 0)
-		(effects
-			(font
-				(size 1.27 1.27)
-				(italic yes)
-			)
-			(justify right bottom)
-		)
-	)
-	(text "IC POWER"
-		(exclude_from_sim no)
-		(at 509.27 77.47 0)
-		(effects
-			(font
-				(size 2.9972 2.9972)
-				(thickness 0.5994)
-				(bold yes)
-			)
-			(justify left bottom)
-		)
-	)
-	(text "FINE"
-		(exclude_from_sim no)
-		(at 87.63 85.725 0)
-		(effects
-			(font
-				(size 1.27 1.27)
-				(italic yes)
-			)
-			(justify right bottom)
-		)
-	)
-	(text "COARSE"
-		(exclude_from_sim no)
-		(at 101.6 283.21 0)
-		(effects
-			(font
-				(size 1.27 1.27)
-				(italic yes)
-			)
-			(justify left bottom)
-		)
-	)
-	(text "POWER HEADER"
-		(exclude_from_sim no)
-		(at 502.92 39.37 0)
-		(effects
-			(font
-				(size 2.9972 2.9972)
-				(thickness 0.5994)
-				(bold yes)
-			)
-			(justify left bottom)
-		)
-	)
-	(text "CONNECTORS\n"
-		(exclude_from_sim no)
-		(at 504.825 191.135 0)
-		(effects
-			(font
-				(size 2.9972 2.9972)
-				(thickness 0.5994)
-				(bold yes)
-			)
-			(justify left bottom)
-		)
-	)
-	(text "VCO2\n"
-		(exclude_from_sim no)
-		(at 353.695 130.81 0)
-		(effects
-			(font
-				(size 2.9972 2.9972)
-				(thickness 0.5994)
-				(bold yes)
-			)
-			(justify right bottom)
-		)
-	)
 	(label "VCO1 SAW OUT"
 		(at 182.245 74.93 0)
-		(fields_autoplaced yes)
 		(effects
 			(font
@@
 	(label "VCO2 PULSE OUT"
 		(at 399.415 170.18 0)
-		(fields_autoplaced yes)
 		(effects
 			(font
@@
 	(label "VCO3 PULSE OUT"
 		(at 196.85 312.42 0)
-		(fields_autoplaced yes)
 		(effects
 			(font
@@
 	(label "VCO2 SAW OUT"
 		(at 400.685 152.4 0)
-		(fields_autoplaced yes)
 		(effects
 			(font
@@
 	(label "VCO1 PULSE OUT"
 		(at 181.61 96.52 0)
-		(fields_autoplaced yes)
 		(effects
 			(font
@@
 	(label "VCO3 SAW OUT"
 		(at 196.215 290.83 0)
-		(fields_autoplaced yes)
 		(effects
 			(font
@@
 	(label "VCO3 MIX OUT"
 		(at 240.665 281.94 0)
-		(fields_autoplaced yes)
 		(effects
 			(font
@@
 		)
 	)
+	(embedded_fonts no)
 )
