File: KiCad/Connector/CONNECTOR.kicad_sch (KiCad schematic)
At the start: 28 parts, among them J1 Conn_01x32_Socket, J10 AudioJack3, J11 AudioJack3, J2 AudioJack3, J3 AudioJack3, J3 Conn_01x32_Socket, J4 AudioJack3, J5 AudioJack3, J6 AudioJack3, J7 AudioJack3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

Commit message: Update BOM
Parts:
- renumbered J9 to J10, J10 to J11, J11 to J12, J3 to J2, J2 to J3, J3 to J4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
